File: hardware/projects/ido/ido.sch (EAGLE design)
At the start: 32 parts, among them U1 PADI-IOT-STAMP, U2 POLOLU-BUCK, U3 AL8805W5, U4 AL8805W5, U5 AL8805W5, X1 PROGRAMMING-HEADER, X10 WIRE-HOLE, X2 UART-HEADER, X3 WIRE-HOLE, X4 WIRE-HOLE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

Commit message: Added debug LEDs.
Parts:
- added LED1, LED2: (no value), led:LEDCHIPLED_0603
- added R4, R5: 261, resistor:R-US_R0603
Connections:
- new net DEBUG1: LED1.A, U1.GA3
- new net DEBUG2: LED2.A, U1.GA5
- new net N$2: LED1.C, R4.2
- new net N$7: LED2.C, R5.2
- net GND: now also R4.1, R5.1
Other:
- moved on the sheet: C1, C2, C3, C4, C5, C6, D1, D2, D3, L1, L2, L3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

Commit message: Preliminary board placement.
Connections:
- removed net N$7: LED2.C, R5.2
- new net N$3: LED2.A, R5.1
- net DEBUG1: now also R4.2; no longer LED1.A
- net DEBUG2: now also R5.2; no longer LED2.A
- net GND: now also LED1.C, LED2.C; no longer R4.1, R5.1
- net N$2: now also LED1.A, R4.1; no longer LED1.C, R4.2
Other:
- moved on the sheet: LED1, LED2, R4, R5
Changed lines of the file:
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@@
 <attribute name="VALUE" x="102.87" y="158.75" size="1.778" layer="96" rot="R180"/>
 </instance>
-<instance part="R4" gate="G$1" x="68.58" y="121.92" smashed="yes" rot="R90">
-<attribute name="NAME" x="69.85" y="124.6886" size="1.778" layer="95"/>
-<attribute name="VALUE" x="66.802" y="119.38" size="1.778" layer="96" rot="R90"/>
+<instance part="R4" gate="G$1" x="68.58" y="132.08" smashed="yes" rot="R90">
+<attribute name="NAME" x="69.85" y="134.8486" size="1.778" layer="95"/>
+<attribute name="VALUE" x="66.802" y="129.54" size="1.778" layer="96" rot="R90"/>
 </instance>
-<instance part="R5" gate="G$1" x="96.52" y="121.92" smashed="yes" rot="R90">
-<attribute name="NAME" x="97.79" y="124.6886" size="1.778" layer="95"/>
-<attribute name="VALUE" x="94.742" y="119.38" size="1.778" layer="96" rot="R90"/>
+<instance part="R5" gate="G$1" x="96.52" y="132.08" smashed="yes" rot="R90">
+<attribute name="NAME" x="97.79" y="134.8486" size="1.778" layer="95"/>
+<attribute name="VALUE" x="94.742" y="129.54" size="1.778" layer="96" rot="R90"/>
 </instance>
-<instance part="LED1" gate="G$1" x="68.58" y="134.62"/>
-<instance part="LED2" gate="G$1" x="96.52" y="134.62"/>
+<instance part="LED1" gate="G$1" x="68.58" y="121.92"/>
+<instance part="LED2" gate="G$1" x="96.52" y="121.92"/>
 <instance part="GND13" gate="1" x="68.58" y="111.76"/>
 <instance part="GND14" gate="1" x="96.52" y="111.76"/>
@@
 </segment>
 <segment>
-<pinref part="R4" gate="G$1" pin="1"/>
+<pinref part="LED1" gate="G$1" pin="C"/>
+<pinref part="GND13" gate="1" pin="GND"/>
 <wire x1="68.58" y1="116.84" x2="68.58" y2="114.3" width="0.1524" layer="91"/>
-<pinref part="GND13" gate="1" pin="GND"/>
-</segment>
-<segment>
-<pinref part="R5" gate="G$1" pin="1"/>
+</segment>
+<segment>
+<pinref part="LED2" gate="G$1" pin="C"/>
+<pinref part="GND14" gate="1" pin="GND"/>
 <wire x1="96.52" y1="116.84" x2="96.52" y2="114.3" width="0.1524" layer="91"/>
-<pinref part="GND14" gate="1" pin="GND"/>
 </segment>
 </net>
@@
 </segment>
 <segment>
-<pinref part="LED1" gate="G$1" pin="A"/>
-<wire x1="68.58" y1="137.16" x2="68.58" y2="139.7" width="0.1524" layer="91"/>
 <wire x1="68.58" y1="139.7" x2="55.88" y2="139.7" width="0.1524" layer="91"/>
 <label x="55.88" y="139.7" size="1.778" layer="95"/>
+<pinref part="R4" gate="G$1" pin="2"/>
+<wire x1="68.58" y1="139.7" x2="68.58" y2="137.16" width="0.1524" layer="91"/>
 </segment>
 </net>
@@
 </segment>
 <segment>
-<pinref part="LED2" gate="G$1" pin="A"/>
-<wire x1="96.52" y1="137.16" x2="96.52" y2="139.7" width="0.1524" layer="91"/>
 <wire x1="96.52" y1="139.7" x2="83.82" y2="139.7" width="0.1524" layer="91"/>
 <label x="83.82" y="139.7" size="1.778" layer="95"/>
+<pinref part="R5" gate="G$1" pin="2"/>
+<wire x1="96.52" y1="139.7" x2="96.52" y2="137.16" width="0.1524" layer="91"/>
 </segment>
 </net>
 <net name="N$2" class="0">
 <segment>
-<pinref part="LED1" gate="G$1" pin="C"/>
-<pinref part="R4" gate="G$1" pin="2"/>
-<wire x1="68.58" y1="129.54" x2="68.58" y2="127" width="0.1524" layer="91"/>
-</segment>
-</net>
-<net name="N$7" class="0">
-<segment>
-<pinref part="LED2" gate="G$1" pin="C"/>
-<pinref part="R5" gate="G$1" pin="2"/>
-<wire x1="96.52" y1="129.54" x2="96.52" y2="127" width="0.1524" layer="91"/>
-</segment>
-</net>
+<pinref part="R4" gate="G$1" pin="1"/>
+<pinref part="LED1" gate="G$1" pin="A"/>
+<wire x1="68.58" y1="127" x2="68.58" y2="124.46" width="0.1524" layer="91"/>
+</segment>
+</net>
+<net name="N$3" class="0">
+<segment>
+<pinref part="R5" gate="G$1" pin="1"/>
+<pinref part="LED2" gate="G$1" pin="A"/>
+<wire x1="96.52" y1="127" x2="96.52" y2="124.46" width="0.1524" layer="91"/>
+</segment>
+</net>

Commit message: Final board rev.
Connections:
- removed net N$2: LED1.A, R4.1
- new net N$5: LED1.C, R4.2
- net DEBUG1: now also LED1.A; no longer R4.2
- net DEBUG2: now also LED2.A; no longer R5.2
- net GND: now also R4.1, R5.1; no longer LED1.C, LED2.C
- net N$3: now also LED2.C, R5.2; no longer LED2.A, R5.1
Other:
- moved on the sheet: LED1, LED2, R4, R5
Changed lines of the file:
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@@
 <setting verticaltext="up"/>
 </settings>
-<grid distance="0.1" unitdist="inch" unit="inch" style="lines" multiple="1" display="yes" altdistance="0.05" altunitdist="inch" altunit="inch"/>
+<grid distance="0.1" unitdist="inch" unit="inch" style="lines" multiple="1" display="no" altdistance="0.01" altunitdist="inch" altunit="inch"/>
 <layers>
 <layer number="1" name="Top" color="4" fill="1" visible="no" active="no"/>
@@
 <attribute name="VALUE" x="102.87" y="158.75" size="1.778" layer="96" rot="R180"/>
 </instance>
-<instance part="R4" gate="G$1" x="68.58" y="132.08" smashed="yes" rot="R90">
-<attribute name="NAME" x="69.85" y="134.8486" size="1.778" layer="95"/>
-<attribute name="VALUE" x="66.802" y="129.54" size="1.778" layer="96" rot="R90"/>
-</instance>
-<instance part="R5" gate="G$1" x="96.52" y="132.08" smashed="yes" rot="R90">
-<attribute name="NAME" x="97.79" y="134.8486" size="1.778" layer="95"/>
-<attribute name="VALUE" x="94.742" y="129.54" size="1.778" layer="96" rot="R90"/>
-</instance>
-<instance part="LED1" gate="G$1" x="68.58" y="121.92"/>
-<instance part="LED2" gate="G$1" x="96.52" y="121.92"/>
+<instance part="R4" gate="G$1" x="68.58" y="121.92" smashed="yes" rot="R90">
+<attribute name="NAME" x="69.85" y="124.6886" size="1.778" layer="95"/>
+<attribute name="VALUE" x="66.802" y="119.38" size="1.778" layer="96" rot="R90"/>
+</instance>
+<instance part="R5" gate="G$1" x="96.52" y="121.92" smashed="yes" rot="R90">
+<attribute name="NAME" x="97.79" y="124.6886" size="1.778" layer="95"/>
+<attribute name="VALUE" x="94.742" y="119.38" size="1.778" layer="96" rot="R90"/>
+</instance>
+<instance part="LED1" gate="G$1" x="68.58" y="134.62"/>
+<instance part="LED2" gate="G$1" x="96.52" y="134.62"/>
 <instance part="GND13" gate="1" x="68.58" y="111.76"/>
 <instance part="GND14" gate="1" x="96.52" y="111.76"/>
@@
 </segment>
 <segment>
-<pinref part="LED1" gate="G$1" pin="C"/>
 <pinref part="GND13" gate="1" pin="GND"/>
+<pinref part="R4" gate="G$1" pin="1"/>
 <wire x1="68.58" y1="116.84" x2="68.58" y2="114.3" width="0.1524" layer="91"/>
 </segment>
 <segment>
-<pinref part="LED2" gate="G$1" pin="C"/>
 <pinref part="GND14" gate="1" pin="GND"/>
+<pinref part="R5" gate="G$1" pin="1"/>
 <wire x1="96.52" y1="116.84" x2="96.52" y2="114.3" width="0.1524" layer="91"/>
 </segment>
@@
 <wire x1="68.58" y1="139.7" x2="55.88" y2="139.7" width="0.1524" layer="91"/>
 <label x="55.88" y="139.7" size="1.778" layer="95"/>
-<pinref part="R4" gate="G$1" pin="2"/>
-<wire x1="68.58" y1="139.7" x2="68.58" y2="137.16" width="0.1524" layer="91"/>
+<pinref part="LED1" gate="G$1" pin="A"/>
+<wire x1="68.58" y1="137.16" x2="68.58" y2="139.7" width="0.1524" layer="91"/>
 </segment>
 </net>
@@
 </segment>
 <segment>
+<pinref part="LED2" gate="G$1" pin="A"/>
+<wire x1="96.52" y1="137.16" x2="96.52" y2="139.7" width="0.1524" layer="91"/>
 <wire x1="96.52" y1="139.7" x2="83.82" y2="139.7" width="0.1524" layer="91"/>
 <label x="83.82" y="139.7" size="1.778" layer="95"/>
+</segment>
+</net>
+<net name="N$3" class="0">
+<segment>
+<pinref part="LED2" gate="G$1" pin="C"/>
 <pinref part="R5" gate="G$1" pin="2"/>
-<wire x1="96.52" y1="139.7" x2="96.52" y2="137.16" width="0.1524" layer="91"/>
-</segment>
-</net>
-<net name="N$2" class="0">
-<segment>
-<pinref part="R4" gate="G$1" pin="1"/>
-<pinref part="LED1" gate="G$1" pin="A"/>
-<wire x1="68.58" y1="127" x2="68.58" y2="124.46" width="0.1524" layer="91"/>
-</segment>
-</net>
-<net name="N$3" class="0">
-<segment>
-<pinref part="R5" gate="G$1" pin="1"/>
-<pinref part="LED2" gate="G$1" pin="A"/>
-<wire x1="96.52" y1="127" x2="96.52" y2="124.46" width="0.1524" layer="91"/>
-</segment>
-</net>
+<wire x1="96.52" y1="129.54" x2="96.52" y2="127" width="0.1524" layer="91"/>
+</segment>
+</net>
+<net name="N$5" class="0">
+<segment>
+<pinref part="LED1" gate="G$1" pin="C"/>
+<pinref part="R4" gate="G$1" pin="2"/>
+<wire x1="68.58" y1="129.54" x2="68.58" y2="127" width="0.1524" layer="91"/>
+</segment>
+</net>
